File: solar_backup_system.sch (EAGLE design)
At the start: 29 parts, among them CON1 5M, CON2 5M, CON3 0.5M, CON4 Anderson, CON5 Anderson, J1 RING-TERMINAL, J2 RING-TERMINAL, X1 5POS

Commit message: removed usb ports
Parts:
- removed USB1, USB2: USB Charger, Dual, bbb:USB-POWER-2
- added CONN1, CONN2, CONN3, CONN4: BARREL-JACK-2.1X5.5MM, aaa:BARREL-JACK-2.1X5.5MM
- added X2, X3: 5POS, bbb:TERMINAL-STRIP-5-3.8MM
- added XJ2, XJ3: TERMINAL-JUMPER-5, bbb:TERMINAL-JUMPER-5
Connections:
- new net N$45: X2-5.1, XJ2-4.2
- new net N$46: X1-5.2, X2-1.2
- new net N$47: X3-5.1, XJ3-4.2
- new net N$48: CIG1.+, FD1.2
- new net N$49: CIG2.+, FD1.3
- new net N$50: FD1.4, X3-1.2
- new net N$51: CIG2.-, X2-4.2
- new net N$52: CIG1.-, X2-5.2
- new net N$53: CONN4.TIP, X3-2.2
- new net N$54: CONN3.TIP, X3-3.2
- new net N$55: CONN2.TIP, X3-4.2
- new net N$56: CONN1.TIP, X3-5.2
- new net N$57: CONN1.RING, X2-3.2
- new net N$59: CONN2.RING, X2-2.2
- new net N$60: CONN3.RING, X1-4.2
- new net N$61: CONN4.RING, X1-3.2
- net N$37: now also X2-1.1, XJ2-1.1; no longer FD1.2, USB1.+
- net N$38: now also X2-2.1, XJ2-1.2, XJ2-2.1; no longer FD1.3, USB2.+
- net N$39: now also X3-1.1, XJ3-1.1; no longer CIG1.+, FD1.4
- net N$40: now also X3-2.1, XJ3-1.2, XJ3-2.1; no longer CIG2.+, FD1.5
- net N$41: now also X3-3.1, XJ3-2.2, XJ3-3.1; no longer CIG2.-, X1-2.2
- net N$42: now also X3-4.1, XJ3-3.2, XJ3-4.1; no longer CIG1.-, X1-3.2
- net N$43: now also X2-3.1, XJ2-2.2, XJ2-3.1; no longer USB2.-, X1-4.2
- net N$44: now also X2-4.1, XJ2-3.2, XJ2-4.1; no longer USB1.-, X1-5.2
Other:
- moved on the sheet: BATT1, CIG1, CIG2, CON1A, CON1B, CON2A, CON2B, CON3A, CON3B, CON4, CON5, F1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
